File: FT232HQ-Xilinx.kicad_pcb (KiCad board)
At the start: 2 copper layers, 30.5 x 20.3 mm, 37 parts, among them J1 USB_C_Receptacle_USB2.0_16P, J2 Conn_01x03_MountingPin, J3 Conn_02x05_Odd_Even, U1 TLV9061xDBV, U3 SN74AVC4T774PW, U4 12M, U5 FT232H, U6 93LCxxBxxOT

Commit message: update
Parts:
- moved U3 0.13 mm to (141.5, 83.1)
Routing:
- net GND: track 15.9 -> 17.4 mm, vias 21 -> 23
- net /TDOR: track 13.4 -> 14.2 mm
- net /TCKR: track 11.3 -> 12.0 mm
- net VREF_F: track 10.8 -> 10.1 mm
- net /EEDIO: track 4.85 -> 4.24 mm

Commit message: update
Parts:
- moved R7 3.47 mm to (136.2, 82.4)
- moved R6 3.35 mm to (136.2, 83.4)
- moved J2 0.18 mm to (129.0, 83.1), turned to 0 degrees
Routing:
- net Net-(J2-Pin_1): track 3.61 -> 8.46 mm
- net +5V: track 49.1 -> 44.4 mm
- net /TCK: track 11.4 -> 6.83 mm, vias 3 -> 2
- net Net-(J2-Pin_3): track 1.79 -> 6.05 mm
- net /TDI: track 9.73 -> 6.00 mm
- net GND: vias 23 -> 24
Other:
- outline, holes or cut-outs redrawn
